File: esquema/dsSpace1104_control.kicad_sch (KiCad schematic)
At the start: 0 parts

Commit message: señal pwm terminada
Parts:
- added C1, C2: 50p, symbol Device:C
- added R1, R2: 270R, symbol Device:R
- added R3, R4: R, symbol Device:R
- added R5: 1K, symbol Device:R
- added R6: 149K, symbol Device:R
- added U1, U2: TC4S584F,LF, Package_TO_SOT_SMD:SOT-23-5, symbol 74xGxx:NC7SVU04P5X
- added U3, U4: H11L1, Package_DIP:DIP-6_W8.89mm_SMDSocket_LongPads, symbol Isolator:H11L1
- added U5: ACS712xLCTR-20A, Package_SO:SOIC-8_3.9x4.9mm_P1.27mm, symbol Sensor_Current:ACS712xLCTR-20A
Connections:
- new net: R5.2, R6.1
- new net: R1.2, U1.2, U3.4
- new net: R2.2, U2.2, U4.4
- new net: U5.1 (IP+), U5.2 (IP+)
- new net: U5.3 (IP-), U5.4 (IP-)
- new net: R3.2, U4.1
- new net: C2.1, U1.4
- new net: R4.2, U3.1
- new net: C1.1, U2.4
- new net +15V: R1.1, R2.1, U1.5 (VCC), U2.5 (VCC), U3.6, U4.6
- new net +5V: U5.8 (VCC)
- new net GND: C1.2, C2.2, R6.2, U1.3 (GND), U2.3 (GND), U3.2, U3.5, U4.2, U4.5, U5.5 (GND)
- new net Vin_750v: R5.1
Other:
- note added: "750V*G=5V"
- note added: "R2/R1=149/1"
