File: esquema/dsSpace1104_control.kicad_sch (KiCad schematic)
At the start: 13 parts, among them U1 TC4S584F,LF, U2 TC4S584F,LF, U3 H11L1, U4 H11L1, U5 ACS712xLCTR-20A

Commit message: filtro segundo grado
Parts:
- added C10, C11, C12, C13, C14, C3, C4, C5, C6, C7, C8, C9: 1u, symbol Device:C
- added R10, R21, R31: 28.7k, symbol Device:R
- added R11, R22, R32: 21.5k, symbol Device:R
- added R12, R15, R20, R25, R30, R35: 1.74k, symbol Device:R
- added R13, R18, R23, R28, R33, R38: 2.49k, symbol Device:R
- added R14, R24, R34: 487, symbol Device:R
- added R16, R26, R36: 1.82k, symbol Device:R
- added R17, R27, R37: 1.37k, symbol Device:R
- added R19, R29, R9: 7.68k, symbol Device:R
- added R39, R40, R41, R42, R7, R8: R, symbol Device:R
- added U10, U11, U8, U9: LM358, symbol Amplifier_Operational:LM358
- added U6: LM358, Package_SO:SOIC-8_3.9x4.9mm_P1.27mm, symbol Amplifier_Operational:LM358
- added U7: ICL7660, Package_SO:SOIC-8_3.9x4.9mm_P1.27mm, symbol Regulator_SwitchedCapacitor:ICL7660
- U5: JLCPCB (none) -> C10681
Connections:
- net +15V: now also U10.8 (V+), U11.8 (V+), U6.8 (V+), U7.8 (V+), U8.8 (V+), U9.8 (V+)
- net GND: now also C11.1, C13.1, C4.1, C5.1, C7.1, C9.1, R10.1, R12.1, R15.1, R16.1, R20.1, R21.1, R25.1, R26.1, R30.1, R31.1, R35.1, R36.1, R40.2, R8.2
- net at R5.2, R6.1: now also U6.3 (+)
- net at U5.7 (VIOUT): now also R39.1
- new net: C8.2, R21.2, U9.3 (+)
- new net: R41.1, R42.2, U6.6 (-)
- new net: R41.2, U6.7
- new net: C5.2, C6.1, R14.2, R17.1
- new net: C6.2, R16.2, U8.5 (+)
- new net: R30.2, R33.1, U10.2 (-)
- new net: R32.2, R33.2, R34.1, U10.1
- new net: C7.2, C8.1, R19.2, R22.1
- new net: R25.2, R28.1, U9.6 (-)
- new net: R27.2, R28.2, U9.7
- new net: C10.1, C9.2, R24.2, R27.1
- new net: C10.2, R26.2, U9.5 (+)
- new net: R39.2, R40.1, U6.5 (+)
- new net: C3.1, C4.2, R11.1, R9.2
- new net: C3.2, R10.2, U8.3 (+)
- new net: C13.2, C14.1, R34.2, R37.1
- new net: C12.2, R31.2, U10.3 (+)
- new net: R11.2, R13.2, R14.1, U8.1
- new net: C11.2, C12.1, R29.2, R32.1
- new net: R7.2, R8.1, U11.3 (+)
- new net: R12.2, R13.1, U8.2 (-)
- new net: R22.2, R23.2, R24.1, U9.1
- new net: R37.2, R38.2, U10.7
- new net: R15.2, R18.1, U8.6 (-)
- new net: R17.2, R18.2, U8.7
- new net: R35.2, R38.1, U10.6 (-)
- new net: R9.1, U11.1, U11.2 (-)
- new net: U6.1, U6.2 (-)
- new net: R20.2, R23.1, U9.2 (-)
- new net: C14.2, R36.2, U10.5 (+)
- new net +2.5V: R42.1
- new net -15V: U10.4 (V-), U11.4 (V-), U6.4 (V-), U7.5 (VOUT), U8.4 (V-), U9.4 (V-)
- new net Vac_400: R7.1
Other:
- note added: "1 de corriete cd 0-20A 1 sensor de tension dc 0-750V 3 sensores de corriente ac de amperios 0-20A 40-200 hz 3 sessores de tension ac de 0-400v 40-200 hz"
- note added: "2.5*g=10V"
- note added: "G=Vin*R2/(R2+R1)"
- note added: "Ideas para laa tenssion ac divisor de tnesion mas fitro paso banda 40-200hz con sallen-key repuesta butterworlf"
- note added: "g=4v/v"
- moved on the sheet: C1, C2, R1, R2, R3, R4, R5, R6, U1, U2, U3, U4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

Commit message: filto intensidad
Parts:
- added C15, C16, C17, C18: 1u, symbol Device:C
- added R43, R44, R45, R46: R, symbol Device:R
- added R47: 21.5k, symbol Device:R
- added R48: 1.37k, symbol Device:R
- added R49: 7.68k, symbol Device:R
- added R50: 487, symbol Device:R
- added R51: 28.7k, symbol Device:R
- added R52: 1.82k, symbol Device:R
- added R53, R55: 1.74k, symbol Device:R
- added R54, R56: 2.49k, symbol Device:R
- added unit 3 of U10
- added U12: ACS712xLCTR-20A, Package_SO:SOIC-8_3.9x4.9mm_P1.27mm, symbol Sensor_Current:ACS712xLCTR-20A
- added U13, U14: LM358, symbol Amplifier_Operational:LM358
- added unit 3 of U9
- R39, R42: value R -> 1k
- R40, R41: value R -> 4k
- R5: value 1K -> 74k
- R6: value 149K -> 1k
Connections:
- net +15V: now also U10.8 (V+), U9.8 (V+); no longer U10.8 (V+), U9.8 (V+)
- net +5V: now also U12.8 (VCC)
- net -15V: now also U10.4 (V-), U9.4 (V-); no longer U10.4 (V-), U9.4 (V-)
- net GND: now also C17.1, C18.1, R44.2, R46.2, R51.1, R52.1, R53.1, R55.1, U12.5 (GND)
- net Vac_400: now also R43.1, R45.1
- net at R19.1: now also U11.6 (-), U11.7
- net at R29.1: now also U13.1, U13.2 (-)
- net at U11.5 (+): now also R43.2, R44.1
- new net: C16.1, C18.2, R48.1, R50.2
- new net: C16.2, R52.2, U14.5 (+)
- new net: U12.1 (IP+), U12.2 (IP+)
- new net: U12.3 (IP-), U12.4 (IP-)
- new net: R49.1, U12.7 (VIOUT)
- new net: R45.2, R46.1, U13.3 (+)
- new net: R48.2, R56.2, U14.7
- new net: R55.2, R56.1, U14.6 (-)
- new net: R47.2, R50.1, R54.2, U14.1
- new net: R53.2, R54.1, U14.2 (-)
- new net: C15.1, C17.2, R47.1, R49.2
- new net: C15.2, R51.2, U14.3 (+)
- no-connect marks 0 -> 2
Other:
- note added: "750V*G=10V"
- note added: "G=1/75"
- note added: "R5/R6=74/1"
- note removed: "750V*G=5V"
- note removed: "G=Vin*R2/(R2+R1)"
- note removed: "R2/R1=149/1"
- moved on the sheet: C10, C11, C12, C13, C14, C3, C4, C5, C6, C7, C8, C9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

Commit message: faltacambiar los conectores a verticales
Parts:
- removed R5: 74k, symbol Device:R
- added C19, C20, C21, C22, C23, C24, C25, C26: 1u, Capacitor_SMD:C_0603_1608Metric_Pad1.08x0.95mm_HandSolder, symbol Device:C
- added C27, C28: 1u, Capacitor_SMD:CP_Elec_4x5.4, symbol Device:C_Polarized
- added J1, J13, J14, J2, J3, J4, J5, J6, J7, J8: Conn_Coaxial, Connector_Coaxial:BNC_Amphenol_B6252HB-NPP3G-50_Horizontal, symbol Connector:Conn_Coaxial
- added J10, J11, J12, J18, J9: Conn_01x02_Socket, Connector:Banana_Jack_2Pin, symbol Connector:Conn_01x02_Socket
- added J15, J16: Conn_01x01_Socket, Connector_PinHeader_2.54mm:PinHeader_1x01_P2.54mm_Vertical, symbol Connector:Conn_01x01_Socket
- added J17: Screw_Terminal_01x02, TerminalBlock_MetzConnect:TerminalBlock_MetzConnect_Type011_RT05502HBLC_1x02_P5.00mm_Horizontal, symbol Connector:Screw_Terminal_01x02
- added R57, R67: 44.2k, symbol Device:R
- added R58, R68: 2.87k, symbol Device:R
- added R59, R69: 7.15k, symbol Device:R
- added R60, R70: 464, symbol Device:R
- added R61, R71: 24.9k, symbol Device:R
- added R62, R72: 1.58k, symbol Device:R
- added R63, R65, R73, R75: 649, symbol Device:R
- added R64, R66, R74, R76: 2.49k, symbol Device:R
- added U15, U17: ACS712xLCTR-20A, Package_SO:SOIC-8_3.9x4.9mm_P1.27mm, symbol Sensor_Current:ACS712xLCTR-20A
- added U16, U18: LM358, Package_SO:SOIC-8_3.9x4.9mm_P1.27mm, symbol Amplifier_Operational:LM358
- added U19: REF3025, Package_TO_SOT_SMD:SOT-23, symbol Reference_Voltage:REF3025
- added U20: L7805, Package_TO_SOT_SMD:TO-252-2, symbol Regulator_Linear:L7805
- C1, C2: footprint (none) -> Capacitor_SMD:C_0603_1608Metric_Pad1.08x0.95mm_HandSolder; JLCPCB (none) -> C1672
- C10, C11, C12, C13, C14, C15, C16, C17, C18, C3, C4, C5, C6, C7, C8, C9: footprint (none) -> Capacitor_SMD:C_0603_1608Metric_Pad1.08x0.95mm_HandSolder; JLCPCB (none) -> C519560
- R1, R2: footprint (none) -> Resistor_SMD:R_0603_1608Metric_Pad0.98x0.95mm_HandSolder; JLCPCB (none) -> C22966
- R3, R4: value R -> 390; footprint (none) -> Resistor_SMD:R_0805_2012Metric_Pad1.20x1.40mm_HandSolder; JLCPCB (none) -> C17655
- R39, R42: footprint (none) -> Resistor_SMD:R_0805_2012Metric_Pad1.20x1.40mm_HandSolder; JLCPCB (none) -> C17513
- R43, R45, R7: value R -> 1k; footprint (none) -> Resistor_SMD:R_0805_2012Metric_Pad1.20x1.40mm_HandSolder; JLCPCB (none) -> C17513
- R44, R46, R8: value R -> 39k
- R47: value 21.5k -> 44.2k
- R48: value 1.37k -> 2.87k
- R49: value 7.68k -> 7.15k
- R50: value 487 -> 464
- R51: value 28.7k -> 24.9k
- R52: value 1.82k -> 1.58k
- R53, R55: value 1.74k -> 649
- R6: value 1k -> 3k; JLCPCB (none) -> C17513
- U10, U11, U13, U14, U8, U9: footprint (none) -> Package_SO:SOIC-8_3.9x4.9mm_P1.27mm; JLCPCB (none) -> C7950
Connections:
- net +15V: now also U13.8 (V+), U14.8 (V+), J17.1 (Pin_1), J18.1 (Pin_1), U16.8 (V+), U18.8 (V+), U20.1 (IN)
- net +2.5V: now also U19.2 (OUT)
- net +5V: now also U15.8 (VCC), U17.8 (VCC)
- net -15V: now also U13.4 (V-), U14.4 (V-), C28.2, U16.4 (V-), U18.4 (V-)
- net GND: now also U7.3 (GND), C21.1, C22.1, C25.1, C26.1, C28.1, J1.2 (Ext), J17.2 (Pin_2), J18.2 (Pin_2), J2.2 (Ext), J3.2 (Ext), J4.2 (Ext), J5.2 (Ext), J6.2 (Ext), J7.2 (Ext), J8.2 (Ext), R61.1, R62.1, R63.1, R65.1, R71.1, R72.1, R73.1, R75.1, U15.5 (GND), U17.5 (GND), U19.3 (GND), U20.2 (GND)
- net Vin_750v: now also U5.3 (IP-), U5.4 (IP-), J9.2 (Pin_2)
- net at R41.2, U6.7: now also J8.1 (In)
- net R_equivalente/SAL_: now reaches R6.1, U6.3 (+)
- net at R27.2, R28.2, U9.7: now also J6.1 (In)
- net at U12.1 (IP+), U12.2 (IP+): now also J10.1 (Pin_1)
- net CH1_Vac_400: now reaches U12.3 (IP-), U12.4 (IP-)
- net CH1_Vac_400: now also R7.1, J10.2 (Pin_2)
- net at R37.2, R38.2, U10.7: now also J7.1 (In)
- net at R17.2, R18.2, U8.7: now also J5.1 (In)
- net at U5.1 (IP+), U5.2 (IP+): now also J9.1 (Pin_1)
- net at R48.2, R56.2, U14.7: now also J2.1 (In)
- net at R3.1: now also J16.1 (Pin_1)
- net at U7.2 (CAP+): now also C27.1
- net at U7.4 (CAP-): now also C27.2
- net at C2.1, U1.4: now also J13.1 (In)
- net at U6.1, U6.2 (-): now also J1.1 (In)
- net at R4.1: now also J15.1 (Pin_1)
- net at C1.1, U2.4: now also J14.1 (In)
- removed net Vac_400: R43.1, R45.1, R7.1
- new net: R73.2, R74.1, U18.2 (-)
- new net: R67.2, R70.1, R74.2, U18.1
- new net: J11.1 (Pin_1), U15.1 (IP+), U15.2 (IP+)
- new net: R75.2, R76.1, U18.6 (-)
- new net: J4.1 (In), R68.2, R76.2, U18.7
- new net: U19.1 (IN), U20.3 (OUT)
- new net: C19.1, C21.2, R57.1, R59.2
- new net: R63.2, R64.1, U16.2 (-)
- new net: R59.1, U15.7 (VIOUT)
- new net: R57.2, R60.1, R64.2, U16.1
- new net: C24.1, C26.2, R68.1, R70.2
- new net: C24.2, R72.2, U18.5 (+)
- new net: R65.2, R66.1, U16.6 (-)
- new net: J3.1 (In), R58.2, R66.2, U16.7
- new net: J12.1 (Pin_1), U17.1 (IP+), U17.2 (IP+)
- new net: C20.1, C22.2, R58.1, R60.2
- new net: C19.2, R61.2, U16.3 (+)
- new net: R69.1, U17.7 (VIOUT)
- new net: C23.1, C25.2, R67.1, R69.2
- new net: C23.2, R71.2, U18.3 (+)
- new net: C20.2, R62.2, U16.5 (+)
- new net CH2_Vac_400: J11.2 (Pin_2), R43.1, U15.3 (IP-), U15.4 (IP-)
- new net CH3_Vac_400: J12.2 (Pin_2), R45.1, U17.3 (IP-), U17.4 (IP-)
- no-connect marks 2 -> 9
Other:
- added sheet R_equivalente (r_equivalente.kicad_sch)
- note added: "2.5W"
- note added: "33.3mw"
- note added: "400V*G=10V"
- note added: "CAMBIAR POR BNC VERTICAL"
- note added: "G=1/40"
- note added: "R1/R2=39/1"
- note added: "R5/R6=(74/1)*3=222/3"
- note removed: "R5/R6=74/1"
- moved on the sheet: C1, C15, C16, C17, C18, C2, R1, R2, R3, R4, R47, R48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

Commit message: bom listo
Parts:
- added R5, R83: 39k, Resistor_SMD:R_2512_6332Metric_Pad1.40x3.35mm_HandSolder, symbol Device:R
- added R84: 2k, Resistor_SMD:R_1206_3216Metric_Pad1.30x1.75mm_HandSolder, symbol Device:R
- R10, R21, R31: footprint (none) -> Resistor_SMD:R_0603_1608Metric_Pad0.98x0.95mm_HandSolder; JLCPCB (none) -> C22928
- R11, R22, R32: footprint (none) -> Resistor_SMD:R_0603_1608Metric_Pad0.98x0.95mm_HandSolder; JLCPCB (none) -> C22911
- R12, R15, R20, R25, R30, R35: footprint (none) -> Resistor_SMD:R_0603_1608Metric_Pad0.98x0.95mm_HandSolder; JLCPCB (none) -> C22848
- R13, R18, R23, R28, R33, R38, R54, R56, R64, R66, R74, R76: footprint (none) -> Resistor_SMD:R_0603_1608Metric_Pad0.98x0.95mm_HandSolder; JLCPCB (none) -> C22908
- R14, R24, R34: footprint (none) -> Resistor_SMD:R_0603_1608Metric_Pad0.98x0.95mm_HandSolder; JLCPCB (none) -> C23064
- R16, R26, R36: footprint (none) -> Resistor_SMD:R_0603_1608Metric_Pad0.98x0.95mm_HandSolder; JLCPCB (none) -> C25958
- R17, R27, R37: footprint (none) -> Resistor_SMD:R_1206_3216Metric_Pad1.30x1.75mm_HandSolder; JLCPCB (none) -> C204642
- R19, R29, R9: footprint (none) -> Resistor_SMD:R_0603_1608Metric_Pad0.98x0.95mm_HandSolder; JLCPCB (none) -> C23102
- R40, R41: footprint (none) -> Resistor_SMD:R_0603_1608Metric_Pad0.98x0.95mm_HandSolder; JLCPCB (none) -> C23040
- R43: value 1k -> 39k; footprint Resistor_SMD:R_0805_2012Metric_Pad1.20x1.40mm_HandSolder -> Resistor_SMD:R_2512_6332Metric_Pad1.40x3.35mm_HandSolder; JLCPCB C17513 -> C7209412
- R44, R46, R8: footprint (none) -> Resistor_SMD:R_2512_6332Metric_Pad1.40x3.35mm_HandSolder; JLCPCB (none) -> C7209412
- R45, R7: value 1k -> 2k; footprint Resistor_SMD:R_0805_2012Metric_Pad1.20x1.40mm_HandSolder -> Resistor_SMD:R_1206_3216Metric_Pad1.30x1.75mm_HandSolder; JLCPCB C17513 -> C17944
- R47, R57, R67: footprint (none) -> Resistor_SMD:R_0603_1608Metric_Pad0.98x0.95mm_HandSolder; JLCPCB (none) -> C23056
- R48, R58, R68: footprint (none) -> Resistor_SMD:R_0603_1608Metric_Pad0.98x0.95mm_HandSolder; JLCPCB (none) -> C22907
- R49, R59, R69: footprint (none) -> Resistor_SMD:R_0603_1608Metric_Pad0.98x0.95mm_HandSolder; JLCPCB (none) -> 0603
- R50, R60, R70: footprint (none) -> Resistor_SMD:R_0603_1608Metric_Pad0.98x0.95mm_HandSolder; JLCPCB (none) -> C23060
- R51, R61, R71: footprint (none) -> Resistor_SMD:R_0603_1608Metric_Pad0.98x0.95mm_HandSolder; JLCPCB (none) -> C25962
- R52, R62, R72: footprint (none) -> Resistor_SMD:R_0603_1608Metric_Pad0.98x0.95mm_HandSolder; JLCPCB (none) -> C22768
- R53, R55, R63, R65, R73, R75: footprint (none) -> Resistor_SMD:R_0805_2012Metric_Pad1.20x1.40mm_HandSolder; JLCPCB (none) -> C17790
- R6: footprint (none) -> Resistor_SMD:R_0805_2012Metric_Pad1.20x1.40mm_HandSolder; JLCPCB C17513 -> C17661
- U6: JLCPCB C5423 -> C7950
Connections:
- net CH1_Vac_400: now also R5.1; no longer R7.1
- net CH3_Vac_400: now also R46.1; no longer R45.1
- net GND: now also R45.2, R7.2, R84.2; no longer R44.2, R46.2, R8.2
- net at R43.2, R44.1: no longer U11.5 (+)
- new net: R44.2, R45.1, U11.5 (+)
- new net: R46.2, R83.1
- new net: R5.2, R8.1
- new net: R7.1, R8.2, U11.3 (+)
- new net: R83.2, R84.1, U13.3 (+)
Other:
- note added: "0.1w"
- note added: "3.9w"
- note added: "78k=1.95"
- moved on the sheet: R8

Commit message: termino enrutamiento falta la filescreem
Parts:
- removed unit 2 of U11
- added C29: 50p, Capacitor_SMD:C_0603_1608Metric_Pad1.08x0.95mm_HandSolder, symbol Device:C
- added J19: Conn_01x01_Socket, Connector_PinHeader_2.54mm:PinHeader_1x01_P2.54mm_Vertical, symbol Connector:Conn_01x01_Socket
- added J20: Conn_Coaxial, proy_lib:Coaxila, symbol Connector:Conn_Coaxial
- added R85: 270R, Resistor_SMD:R_0603_1608Metric_Pad0.98x0.95mm_HandSolder, symbol Device:R
- added R86: 390, Resistor_SMD:R_0805_2012Metric_Pad1.20x1.40mm_HandSolder, symbol Device:R
- added unit 1 of U11
- added U21: H11L1, Package_DIP:DIP-6_W8.89mm_SMDSocket_LongPads, symbol Isolator:H11L1
- added U22: TC4S584F,LF, Package_TO_SOT_SMD:SOT-23-5, symbol 74xGxx:NC7SVU04P5X
- added U23: LM358, Package_SO:SOIC-8_3.9x4.9mm_P1.27mm, symbol Amplifier_Operational:LM358
- J1, J13, J14, J2, J3, J4, J5, J6, J7, J8: footprint Connector_Coaxial:BNC_Amphenol_B6252HB-NPP3G-50_Horizontal -> proy_lib:Coaxila
Connections:
- net +15V: now also R85.1, U21.6, U22.5 (VCC), U23.8 (V+)
- net +5V: now also U19.1 (IN), U20.3 (OUT)
- net -15V: now also U23.4 (V-)
- net GND: now also J13.2 (Ext), J14.2 (Ext), C29.2, J20.2 (Ext), U21.2, U21.5, U22.3 (GND)
- net POT3: now reaches J11.1 (Pin_1), U15.1 (IP+), U15.2 (IP+)
- net at R19.1: now also U23.1, U23.2 (-)
- net at R44.2, R45.1: now also U23.3 (+)
- net POT2: now reaches J10.1 (Pin_1), U12.1 (IP+), U12.2 (IP+)
- net POT4: now reaches J12.1 (Pin_1), U17.1 (IP+), U17.2 (IP+)
- net POT1: now reaches J9.1 (Pin_1), U5.1 (IP+), U5.2 (IP+)
- net at R7.1, R8.2: now also U11.3 (+); no longer U11.3 (+)
- new net: C29.1, J20.1 (In), U22.4
- new net: J19.1 (Pin_1), R86.1
- new net: R85.2, U21.4, U22.2
- new net: R86.2, U21.1
- new net: R9.1, U11.1, U11.2 (-)
- no-connect marks 9 -> 15
Other:
- moved on the sheet: C1, C10, C11, C12, C13, C14, C15, C16, C17, C18, C19, C2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

Commit message: mando fabrica
Parts:
- AC_I_CH1: renamed from J2; footprint proy_lib:Coaxila -> Connector_Coaxial:SMA_Amphenol_901-144_Vertical; JLCPCB C709673 -> C496549
- AC_I_CH2: renamed from J3; footprint proy_lib:Coaxila -> Connector_Coaxial:SMA_Amphenol_901-144_Vertical; JLCPCB C709673 -> C496549
- AC_I_CH3: renamed from J4; footprint proy_lib:Coaxila -> Connector_Coaxial:SMA_Amphenol_901-144_Vertical; JLCPCB C709673 -> C496549
- AC_V_CH2: renamed from J6; footprint proy_lib:Coaxila -> Connector_Coaxial:SMA_Amphenol_901-144_Vertical; JLCPCB C709673 -> C496549
- AC_V_CH3: renamed from J7; footprint proy_lib:Coaxila -> Connector_Coaxial:SMA_Amphenol_901-144_Vertical; JLCPCB C709673 -> C496549
- A_V_CH1: renamed from J5; footprint proy_lib:Coaxila -> Connector_Coaxial:SMA_Amphenol_901-144_Vertical; JLCPCB C709673 -> C496549
- DC_I1: renamed from J8; footprint proy_lib:Coaxila -> Connector_Coaxial:SMA_Amphenol_901-144_Vertical; JLCPCB C709673 -> C496549
- DC_V1: renamed from J1; footprint proy_lib:Coaxila -> Connector_Coaxial:SMA_Amphenol_901-144_Vertical; JLCPCB C709673 -> C496549
- PWM1: renamed from J20; footprint proy_lib:Coaxila -> Connector_Coaxial:SMA_Amphenol_901-144_Vertical; JLCPCB C709673 -> C496549
- PWM2: renamed from J13; footprint proy_lib:Coaxila -> Connector_Coaxial:SMA_Amphenol_901-144_Vertical; JLCPCB C709673 -> C496549
- PWM3: renamed from J14; footprint proy_lib:Coaxila -> Connector_Coaxial:SMA_Amphenol_901-144_Vertical; JLCPCB C709673 -> C496549
- U7: JLCPCB C19193423 -> C28595
