File: esquema/r_equivalente.kicad_sch (KiCad schematic)
At the start: 6 parts

Commit message: bom listo
Parts:
- R80: footprint (none) -> Resistor_SMD:R_1206_3216Metric_Pad1.30x1.75mm_HandSolder; JLCPCB (none) -> C17944
Changed lines of the file:
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@@
 			)
 		)
-		(property "Footprint" ""
+		(property "Footprint" "Resistor_SMD:R_1206_3216Metric_Pad1.30x1.75mm_HandSolder"
 			(at 132.842 68.58 90)
 			(effects
@@
 			)
 		)
-		(property "Datasheet" "~"
+		(property "Datasheet" "https://jlcpcb.com/partdetail/18632-1206W4F2001T5E/C17944"
 			(at 134.62 68.58 0)
 			(effects
@@
 			(at 134.62 68.58 0)
 			(effects
+				(font
+					(size 1.27 1.27)
+				)
+				(hide yes)
+			)
+		)
+		(property "JLCPCB" "C17944"
+			(at 134.62 68.58 0)
+			(effects
