File: esquema/dsSpace1104_control.kicad_pcb (KiCad board)
At the start: 4 copper layers, 140.3 x 128 mm, 158 parts, among them J1 Conn_Coaxial, J10 Conn_01x02_Socket, J11 Conn_01x02_Socket, J12 Conn_01x02_Socket, J13 Conn_Coaxial, J14 Conn_Coaxial, J15 Conn_01x01_Socket, J16 Conn_01x01_Socket, J17 Screw_Terminal_01x02, J18 Conn_01x02_Socket, J19 Conn_01x01_Socket, J2 Conn_Coaxial, J20 Conn_Coaxial, J3 Conn_Coaxial, J4 Conn_Coaxial, J5 Conn_Coaxial, J6 Conn_Coaxial, J7 Conn_Coaxial, J8 Conn_Coaxial, J9 Conn_01x02_Socket, U1 TC4S584F,LF, U10 LM358, U11 LM358, U12 ACS712xLCTR-20A, U13 LM358, U14 LM358, U15 ACS712xLCTR-20A, U16 LM358, U17 ACS712xLCTR-20A, U18 LM358, U19 REF3025, U2 TC4S584F,LF, U20 L7805, U21 H11L1, U22 TC4S584F,LF, U23 LM358, U3 H11L1, U4 H11L1, U5 ACS712xLCTR-20A, U6 LM358, U7 ICL7660, U8 LM358, U9 LM358

Commit message: serigrafia terminada
Parts:
- moved PWM2 0.32 mm to (121.8, 60.2)
- renumbered J2 to AC_I_CH1, J3 to AC_I_CH2, J4 to AC_I_CH3, J6 to AC_V_CH2, J7 to AC_V_CH3, J8 to DC_I, J1 to DC_V, J5 to JAC_V_CH1, J14 to PWM1, J13 to PWM2, J20 to PWM3
Changed lines of the file:
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@@
 		(tags "resistor handsolder")
 		(property "Reference" "R37"
-			(at 4.064 0 90)
+			(at -0.609 2.557 90)
 			(layer "B.SilkS")
 			(effects
@@
 		(tags "SOIC SO")
 		(property "Reference" "U23"
-			(at 2.5 3.925 90)
+			(at 3.675 -3.3 90)
 			(layer "B.SilkS")
 			(effects
@@
 		(tags "THT terminal block Metz Connect Type011_RT05502HBLC pitch 5mm size 10x10.5mm drill 1.4mm pad 2.8mm")
 		(property "Reference" "J17"
-			(at -15.28 -1.1685 0)
+			(at 11.759 1.1895 0)
 			(layer "B.SilkS")
 			(effects
@@
 		(tags "resistor handsolder")
 		(property "Reference" "R56"
-			(at 0 1.43 0)
+			(at 3.215 0.0375 0)
 			(layer "B.SilkS")
 			(effects
@@
 		(layer "B.Cu")
 		(at 111.025 118.805 180)
-		(property "Reference" "J5"
-			(at -5.0625 0.715 0)
+		(property "Reference" "JAC_V_CH1"
+			(at 0 -9.295 0)
 			(unlocked yes)
 			(layer "B.SilkS")
@@
 		(layer "B.Cu")
 		(at 133.01 88.28 180)
-		(property "Reference" "J7"
-			(at -0.15 0.715 0)
+		(property "Reference" "AC_V_CH3"
+			(at -0.09 -9.62 0)
 			(unlocked yes)
 			(layer "B.SilkS")
@@
 		)
 		(fp_text user "${REFERENCE}"
-			(at -0.15 -2.285 0)
+			(at 0.085 -9.095 0)
 			(unlocked yes)
 			(layer "B.Fab")
@@
 		(tags "banana socket")
 		(property "Reference" "J10"
-			(at 14.985 6.24 0)
+			(at 14.895 0.01 0)
 			(layer "B.SilkS")
 			(effects
@@
 		(tags "resistor handsolder")
 		(property "Reference" "R34"
-			(at -3.556 0 90)
+			(at 0.059 2.228 90)
 			(layer "B.SilkS")
 			(effects
@@
 		(tags "banana socket")
 		(property "Reference" "J18"
-			(at 14.985 6.24 0)
+			(at 15.204 0.106 0)
 			(layer "B.SilkS")
 			(effects
@@
 		(layer "B.Cu")
 		(at 92.525 118.89 180)
-		(property "Reference" "J2"
-			(at -5.0625 0.715 0)
+		(property "Reference" "AC_I_CH1"
+			(at 0.05 -8.96 0)
 			(unlocked yes)
 			(layer "B.SilkS")
@@
 		(tags "banana socket")
 		(property "Reference" "J11"
-			(at 14.985 6.24 0)
+			(at 14.97 -0.015 0)
 			(layer "B.SilkS")
 			(effects
@@
 		(tags "banana socket")
 		(property "Reference" "J12"
-			(at 14.985 6.24 90)
+			(at 15.37 -0.05 90)
 			(layer "B.SilkS")
 			(effects
@@
 		(layer "B.Cu")
 		(at 152.005 118.805 180)
-		(property "Reference" "J3"
-			(at -0.15 0.715 0)
+		(property "Reference" "AC_I_CH2"
+			(at 0.005 -9.07 0)
 			(unlocked yes)
 			(layer "B.SilkS")
@@
 		)
 		(fp_text user "${REFERENCE}"
-			(at -0.15 -2.285 0)
+			(at 0.03 -8.72 0)
 			(unlocked yes)
 			(layer "B.Fab")
@@
 		(tags "resistor handsolder")
 		(property "Reference" "R18"
-			(at 0 -1.475 90)
+			(at -0.025 -1.4875 90)
 			(layer "B.SilkS")
 			(effects
@@
 	(footprint "proy_lib:Coaxila"
 		(layer "B.Cu")
-		(at 121.85 59.85 180)
-		(property "Reference" "J13"
-			(at -0.15 0.715 0)
+		(at 121.78 60.165 180)
+		(property "Reference" "PWM2"
+			(at 0.13 -9.885 0)
 			(unlocked yes)
 			(layer "B.SilkS")
@@
 			(layer "B.Fab")
 		)
-		(fp_text user "${REFERENCE}"
-			(at -0.15 -2.285 0)
+		(fp_text user "PWM2"
+			(at -0.045 -9.01 0)
 			(unlocked yes)
 			(layer "B.Fab")
@@
 		(layer "B.Cu")
 		(at 92.505 88.18 180)
-		(property "Reference" "J8"
-			(at -0.15 0.715 0)
+		(property "Reference" "DC_I"
+			(at -0.195 -9.345 0)
 			(unlocked yes)
 			(layer "B.SilkS")
@@
 		)
 		(property "Value" "Conn_Coaxial"
-			(at -0.15 -0.785 0)
+			(at -2.17 -12.095 0)
 			(unlocked yes)
 			(layer "B.Fab")
@@
 		)
 		(fp_text user "${REFERENCE}"
-			(at -0.15 -2.285 0)
+			(at 0.005 -9.845 0)
 			(unlocked yes)
 			(layer "B.Fab")
@@
 		(layer "B.Cu")
 		(at 152.005 88.39 180)
-		(property "Reference" "J4"
-			(at -0.15 0.715 0)
+		(property "Reference" "AC_I_CH3"
+			(at -0.02 -9.485 0)
 			(unlocked yes)
-			(layer "F.SilkS")
+			(layer "B.SilkS")
 			(effects
 				(font
@@
 					(thickness 0.1)
 				)
+				(justify mirror)
 			)
 		)
@@
 		)
 		(fp_text user "${REFERENCE}"
-			(at -0.15 -2.285 0)
+			(at -0.295 -8.535 0)
 			(unlocked yes)
 			(layer "B.Fab")
@@
 		(tags "banana socket")
 		(property "Reference" "J9"
-			(at 14.985 6.24 90)
+			(at 17.71 0.005 90)
 			(layer "B.SilkS")
 			(effects
@@
 		(layer "B.Cu")
 		(at 103.83 60.115 180)
-		(property "Reference" "J20"
-			(at -0.15 0.715 0)
+		(property "Reference" "PWM3"
+			(at 0.205 -10.41 0)
 			(unlocked yes)
 			(layer "B.SilkS")
@@
 		)
 		(fp_text user "${REFERENCE}"
-			(at -0.15 -2.285 0)
+			(at -0.02 -9.06 0)
 			(unlocked yes)
 			(layer "B.Fab")
@@
 		(layer "B.Cu")
 		(at 111.025 88.305 180)
-		(property "Reference" "J1"
-			(at -0.15 0.715 0)
+		(property "Reference" "DC_V"
+			(at -0.025 -9.395 0)
 			(unlocked yes)
 			(layer "B.SilkS")
@@
 		)
 		(fp_text user "${REFERENCE}"
-			(at -0.15 -2.285 0)
+			(at 0.025 -9.545 0)
 			(unlocked yes)
 			(layer "B.Fab")
@@
 		(layer "B.Cu")
 		(at 139.68 60.24 180)
-		(property "Reference" "J14"
-			(at -0.15 0.715 180)
+		(property "Reference" "PWM1"
+			(at -0.12 -9.935 0)
 			(unlocked yes)
-			(layer "F.SilkS")
+			(layer "B.SilkS")
 			(effects
 				(font
@@
 		)
 		(fp_text user "${REFERENCE}"
-			(at -0.15 -2.285 0)
+			(at 0.28 -9.485 0)
 			(unlocked yes)
 			(layer "B.Fab")
@@
 		(layer "B.Cu")
 		(at 133.375 118.805 180)
-		(property "Reference" "J6"
-			(at -0.15 0.715 0)
+		(property "Reference" "AC_V_CH2"
+			(at 0.05 -9.17 0)
 			(unlocked yes)
 			(layer "B.SilkS")
@@
 		)
 		(fp_text user "${REFERENCE}"
-			(at -0.15 -2.285 0)
+			(at 0.15 -2.87 0)
 			(unlocked yes)
 			(layer "B.Fab")
@@
 	)
 	(segment
-		(start 110.0481 134.1703)
+		(start 109.4877 134.1703)
 		(end 107.4797 134.1703)
 		(width 0.2)
@@
 	)
 	(segment
-		(start 110.0481 134.1703)
-		(end 110.1949 134.1703)
+		(start 110.4131 134.3885)
+		(end 111.6589 134.3885)
 		(width 0.2)
 		(layer "B.Cu")
@@
 	)
 	(segment
-		(start 107.4797 134.1703)
-		(end 106.65 135)
+		(start 110.0481 134.0235)
+		(end 110.4131 134.3885)
 		(width 0.2)
 		(layer "B.Cu")
@@
 	)
 	(segment
-		(start 113.3125 136.0421)
-		(end 113.3125 136.45)
+		(start 111.6589 134.3885)
+		(end 113.3125 136.0421)
 		(width 0.2)
 		(layer "B.Cu")
@@
 	(segment
 		(start 110.0481 133.6099)
-		(end 110.0481 134.1703)
+		(end 109.4877 134.1703)
 		(width 0.2)
 		(layer "B.Cu")
@@
 	)
 	(segment
-		(start 110.1949 134.1703)
-		(end 110.4131 134.3885)
+		(start 110.0481 133.6099)
+		(end 110.0481 134.0235)
 		(width 0.2)
 		(layer "B.Cu")
@@
 	)
 	(segment
-		(start 111.6589 134.3885)
-		(end 113.3125 136.0421)
+		(start 113.3125 136.0421)
+		(end 113.3125 136.45)
 		(width 0.2)
 		(layer "B.Cu")
@@
 	)
 	(segment
-		(start 110.4131 134.3885)
-		(end 111.6589 134.3885)
+		(start 107.4797 134.1703)
+		(end 106.65 135)
 		(width 0.2)
 		(layer "B.Cu")

Commit message: mando fabrica
Parts:
- AC_I_CH1, AC_I_CH2, AC_I_CH3, AC_V_CH2, AC_V_CH3, PWM2: footprint proy_lib:Coaxila -> Connector_Coaxial:SMA_Amphenol_901-144_Vertical
- A_V_CH1: renamed from JAC_V_CH1; footprint proy_lib:Coaxila -> Connector_Coaxial:SMA_Amphenol_901-144_Vertical
- DC_I1: renamed from DC_I; footprint proy_lib:Coaxila -> Connector_Coaxial:SMA_Amphenol_901-144_Vertical
- DC_V1: renamed from DC_V; footprint proy_lib:Coaxila -> Connector_Coaxial:SMA_Amphenol_901-144_Vertical
- PWM1: renamed from PWM3; footprint proy_lib:Coaxila -> Connector_Coaxial:SMA_Amphenol_901-144_Vertical
- PWM3: renamed from PWM1; footprint proy_lib:Coaxila -> Connector_Coaxial:SMA_Amphenol_901-144_Vertical
- R29, U13: moved to B.Cu
- moved C14 75.0 mm to (208.7, 114.2), turned to 90 degrees
- moved R31 74.2 mm to (208.7, 118.5), turned to 90 degrees
- moved R36 72.5 mm to (205.9, 109.7), turned to -90 degrees
- moved C11 71.9 mm to (207.1, 124.3), turned to -90 degrees
- moved R35 69.4 mm to (203.6, 109.7), turned to -90 degrees
- moved C12 69.3 mm to (205.3, 124.3), turned to 90 degrees
- moved R37 68.5 mm to (204.1, 114.7), turned to 180 degrees
- moved U10 68.2 mm to (204.1, 115.9), turned to 90 degrees
- moved R34 68.0 mm to (204.1, 117.2), turned to 0 degrees
- moved R30 66.8 mm to (203.6, 124.3), turned to 90 degrees
- moved R38 66.6 mm to (201.5, 109.6), turned to -90 degrees
- moved R33 66.1 mm to (203.1, 121.0), turned to 180 degrees
- moved C13 63.9 mm to (201.5, 124.2), turned to 90 degrees
- moved R29 63.0 mm to (209.8, 126.5)
- moved R32 62.0 mm to (200.0, 119.1), turned to 90 degrees
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Routing:
- net Net-(DC_V1-In): track 54.1 -> 73.6 mm
- net Net-(DC_I1-In): track 21.6 -> 37.7 mm
- net Net-(AC_V_CH3-In): track 34.3 -> 19.3 mm, vias 1 -> 2
- net -15V: track 20.2 -> 33.0 mm
- net +15V: track 66.3 -> 56.9 mm, vias 12 -> 11
- net Net-(AC_I_CH3-In): track 25.6 -> 31.2 mm
- net Net-(C11-Pad2): track 24.6 -> 21.1 mm, vias 0 -> 1
- net Net-(R43-Pad2): track 11.6 -> 15.0 mm
- net Net-(U13A-+): track 11.2 -> 7.80 mm, vias 0 -> 1
- net Net-(R46-Pad2): track 7.48 -> 5.13 mm
- net /+2.5V: track 8.47 -> 10.6 mm
- net Net-(R32-Pad2): track 8.61 -> 7.45 mm
- net GND: track 24.0 -> 22.9 mm, vias 13 -> 12
- net Net-(U17-VIOUT): track 15.6 -> 16.6 mm, vias 0 -> 2
- net Net-(U12-VIOUT): track 7.68 -> 8.39 mm
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- added copper zone on In1.Cu, net /CH1_Vac_400
- added copper zone on In2.Cu, net /CH1_Vac_400
- added copper zone on In1.Cu, net /CH2_Vac_400
- added copper zone on In2.Cu, net /CH2_Vac_400
- added copper zone on In1.Cu, net /CH3_Vac_400
- added copper zone on In2.Cu, net /CH3_Vac_400
- added copper zone on In1.Cu, net /POT1
- added copper zone on In2.Cu, net /POT1
- added copper zone on In1.Cu, net /POT2
- added copper zone on In2.Cu, net /POT2
- added copper zone on In1.Cu, net /POT3
- added copper zone on In2.Cu, net /POT3
- added copper zone on In1.Cu, net /POT4
- added copper zone on In2.Cu, net /POT4
- added copper zone on In1.Cu, net /Vin_750v
- added copper zone on In2.Cu, net /Vin_750v
Other:
- board size 140.3 x 128 mm -> 164.9 x 128 mm
